File: kicad/fan.kicad_sch (KiCad schematic)
At the start: 5 parts, among them M1 Fan_Tacho_PWM, Q1 2N7000, Q2 2N7000

Commit message: basic layout
Connections:
- net PWM: now also Q2.2 (G); no longer M1.4 (PWM), Q2.3 (D), R3.2
- new net: M1.4 (PWM), Q2.3 (D), R3.2
Changed lines of the file:
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@@
 	(wire
 		(pts
-			(xy 132.08 104.14) (xy 67.31 104.14)
+			(xy 67.31 109.22) (xy 124.46 109.22)
 		)
 		(stroke
@@
 		)
 	)
-	(wire
-		(pts
-			(xy 67.31 104.14) (xy 67.31 105.41)
-		)
-		(stroke
-			(width 0)
-			(type default)
-		)
-	)
 	(rectangle
 		(start 106.68 69.85)
@@
 	(hierarchical_label "PWM"
 		(shape input)
-		(at 67.31 105.41 180)
+		(at 67.31 109.22 180)
 		(fields_autoplaced yes)
 		(effects

Commit message: revA
Parts:
- removed Q1, Q2: 2N7000, Package_TO_SOT_THT:TO-92_Inline, symbol Transistor_FET:2N7000
- added Q1, Q9: 2N7002, Package_TO_SOT_SMD:SOT-23, symbol Transistor_FET:2N7002
Connections:
- net GND: now also Q1.2 (S), Q9.2 (S)
- net PWM: now also Q1.1 (G)
- net TACHO: now also Q9.3 (D)
- net at M1.3 (Tacho): now also Q9.1 (G)
- net at M1.4 (PWM), R3.2: now also Q1.3 (D)
Changed lines of the file:
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@@
+	)
+	(symbol
+		(lib_id "Transistor_FET:2N7002")
+		(at 129.54 109.22 0)
+		(unit 1)
+		(exclude_from_sim no)
+		(in_bom yes)
+		(on_board yes)
+		(dnp no)
+		(fields_autoplaced yes)
+		(property "Reference" "Q1"
+			(at 135.89 107.9499 0)
+			(effects
+				(font
+					(size 1.27 1.27)
+				)
+				(justify left)
+			)
+		)
+		(property "Value" "2N7002"
+			(at 135.89 110.4899 0)
+			(effects
+				(font
+					(size 1.27 1.27)
+				)
+				(justify left)
+			)
+		)
+		(property "Footprint" "Package_TO_SOT_SMD:SOT-23"
+			(at 134.62 111.125 0)
+			(effects
+				(font
+					(size 1.27 1.27)
+					(italic yes)
+				)
+				(justify left)
+				(hide yes)
+			)
+		)
+		(property "Datasheet" "https://www.onsemi.com/pub/Collateral/NDS7002A-D.PDF"
+			(at 134.62 113.03 0)
+			(effects
+				(font
+					(size 1.27 1.27)
+				)
+				(justify left)
+				(hide yes)
+			)
+		)
+		(property "Description" "0.115A Id, 60V Vds, N-Channel MOSFET, SOT-23"
+			(at 129.54 109.22 0)
+			(effects
+				(font
+					(size 1.27 1.27)
+				)
+				(hide yes)
+			)
+		)
+		(pin "3"
+		)
+		(pin "2"
+		)
+		(pin "1"
+		)
+		(instances
+			(project "multifan-i2c-controller"
+				(path "/a9a5da40-a42e-45e4-ab10-820f7b034c24/31b761fd-990f-4530-8b3a-6741ab18454d"
+					(reference "Q1")
+					(unit 1)
+				)
+				(path "/a9a5da40-a42e-45e4-ab10-820f7b034c24/be8049d5-6f29-4d60-8441-bb89437ffa26"
+					(reference "Q2")
+					(unit 1)
+				)
+				(path "/a9a5da40-a42e-45e4-ab10-820f7b034c24/da56f3fa-ae89-4bf3-a7d8-c42abaec7938"
+					(reference "Q3")
+					(unit 1)
+				)
+				(path "/a9a5da40-a42e-45e4-ab10-820f7b034c24/75bddcd0-0fc4-4a51-b004-02588bb9cb75"
+					(reference "Q4")
+					(unit 1)
+				)
+			)
+		)
 	)
 	(symbol
@@
 	)
 	(symbol
-		(lib_id "Transistor_FET:2N7000")
-		(at 129.54 109.22 0)
-		(unit 1)
-		(exclude_from_sim no)
-		(in_bom yes)
-		(on_board yes)
-		(dnp no)
-		(fields_autoplaced yes)
-		(property "Reference" "Q2"
-			(at 135.89 107.9499 0)
-			(effects
-				(font
-					(size 1.27 1.27)
-				)
-				(justify left)
-			)
-		)
-		(property "Value" "2N7000"
-			(at 135.89 110.4899 0)
-			(effects
-				(font
-					(size 1.27 1.27)
-				)
-				(justify left)
-			)
-		)
-		(property "Footprint" "Package_TO_SOT_THT:TO-92_Inline"
-			(at 134.62 111.125 0)
-			(effects
-				(font
-					(size 1.27 1.27)
-					(italic yes)
-				)
-				(justify left)
-				(hide yes)
-			)
-		)
-		(property "Datasheet" "https://www.vishay.com/docs/70226/70226.pdf"
-			(at 134.62 113.03 0)
-			(effects
-				(font
-					(size 1.27 1.27)
-				)
-				(justify left)
-				(hide yes)
-			)
-		)
-		(property "Description" "0.2A Id, 200V Vds, N-Channel MOSFET, 2.6V Logic Level, TO-92"
-			(at 129.54 109.22 0)
-			(effects
-				(font
-					(size 1.27 1.27)
-				)
-				(hide yes)
-			)
-		)
-		(pin "1"
-		)
-		(pin "3"
-		)
-		(pin "2"
-		)
-		(instances
-			(project "multifan-i2c-controller"
-				(path "/a9a5da40-a42e-45e4-ab10-820f7b034c24/31b761fd-990f-4530-8b3a-6741ab18454d"
-					(reference "Q2")
-					(unit 1)
-				)
-				(path "/a9a5da40-a42e-45e4-ab10-820f7b034c24/be8049d5-6f29-4d60-8441-bb89437ffa26"
-					(reference "Q4")
-					(unit 1)
-				)
-				(path "/a9a5da40-a42e-45e4-ab10-820f7b034c24/da56f3fa-ae89-4bf3-a7d8-c42abaec7938"
-					(reference "Q6")
-					(unit 1)
-				)
-				(path "/a9a5da40-a42e-45e4-ab10-820f7b034c24/75bddcd0-0fc4-4a51-b004-02588bb9cb75"
-					(reference "Q8")
-					(unit 1)
-				)
-			)
-		)
-	)
-	(symbol
-		(lib_id "Transistor_FET:2N7000")
+		(lib_id "Transistor_FET:2N7002")
 		(at 121.92 88.9 0)
 		(mirror y)
@@
 		(on_board yes)
 		(dnp no)
-		(property "Reference" "Q1"
+		(property "Reference" "Q9"
 			(at 115.57 87.6299 0)
 			(effects
@@
 			)
 		)
-		(property "Value" "2N7000"
+		(property "Value" "2N7002"
 			(at 115.57 90.1699 0)
 			(effects
@@
 			)
 		)
-		(property "Footprint" "Package_TO_SOT_THT:TO-92_Inline"
+		(property "Footprint" "Package_TO_SOT_SMD:SOT-23"
 			(at 116.84 90.805 0)
 			(effects
@@
 			)
 		)
-		(property "Datasheet" "https://www.vishay.com/docs/70226/70226.pdf"
+		(property "Datasheet" "https://www.onsemi.com/pub/Collateral/NDS7002A-D.PDF"
 			(at 116.84 92.71 0)
 			(effects
@@
 			)
 		)
-		(property "Description" "0.2A Id, 200V Vds, N-Channel MOSFET, 2.6V Logic Level, TO-92"
+		(property "Description" "0.115A Id, 60V Vds, N-Channel MOSFET, SOT-23"
 			(at 121.92 88.9 0)
 			(effects
@@
 			)
 		)
+		(pin "3"
+		)
+		(pin "2"
+		)
 		(pin "1"
-		)
-		(pin "3"
-		)
-		(pin "2"
 		)
 		(instances
 			(project "multifan-i2c-controller"
 				(path "/a9a5da40-a42e-45e4-ab10-820f7b034c24/31b761fd-990f-4530-8b3a-6741ab18454d"
-					(reference "Q1")
+					(reference "Q9")
 					(unit 1)
 				)
 				(path "/a9a5da40-a42e-45e4-ab10-820f7b034c24/be8049d5-6f29-4d60-8441-bb89437ffa26"
-					(reference "Q3")
+					(reference "Q10")
 					(unit 1)
 				)
 				(path "/a9a5da40-a42e-45e4-ab10-820f7b034c24/da56f3fa-ae89-4bf3-a7d8-c42abaec7938"
-					(reference "Q5")
+					(reference "Q11")
 					(unit 1)
 				)
 				(path "/a9a5da40-a42e-45e4-ab10-820f7b034c24/75bddcd0-0fc4-4a51-b004-02588bb9cb75"
-					(reference "Q7")
-					(unit 1)
-				)
+					(reference "Q12")
+					(unit 1)
+				)
