File: kicad/multifan-i2c-controller.kicad_pcb (KiCad board)
At the start: 2 copper layers, 66 x 91.4 mm, 43 parts, among them J2 Conn_01x02, J4 AVR-ISP-6, M1 Fan_Tacho_PWM, M2 Fan_Tacho_PWM, M3 Fan_Tacho_PWM, M4 Fan_Tacho_PWM, Q1 2N7000, Q2 2N7000, Q3 2N7000, Q4 2N7000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

Commit message: basic layout
Parts:
- added J1: I2C, Connector_Molex:Molex_KK-254_AE-6410-04A_1x04_P2.54mm_Vertical, F.Cu at (140.3, 152.4)
- added SW1: SW_Push, Button_Switch_SMD:SW_Push_1P1T_NO_6x6mm_H9.5mm, F.Cu at (139.9, 75.9)
- added Y1: 16M, Crystal:Crystal_HC49-U_Vertical, F.Cu at (108.0, 135.8)
- moved R13 125.8 mm to (89.5, 160.7), turned to 180 degrees
- moved R12 123.1 mm to (90.2, 154.3), turned to 180 degrees
- moved C1 119.7 mm to (100.0, 138.4)
- moved D1 117.4 mm to (83.9, 157.7)
- moved D2 117.4 mm to (83.9, 161.1)
- moved C5 112.4 mm to (131.4, 164.5)
- moved C2 110.9 mm to (100.0, 128.3), turned to 180 degrees
- moved C3 110.4 mm to (139.7, 163.2)
- moved R1 107.2 mm to (101.6, 133.3), turned to -90 degrees
- moved Q4 104.4 mm to (103.5, 119.7)
- moved R4 103.0 mm to (112.4, 112.4)
- moved R5 103.0 mm to (112.4, 115.7)
- moved Q3 102.6 mm to (104.1, 110.8)
- moved R11 87.6 mm to (133.3, 139.7), turned to -90 degrees
- moved R10 87.6 mm to (139.7, 139.7), turned to -90 degrees
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Connections:
- M1 pad 4: /fan/PWM -> Net-(M1-PWM)
- M2 pad 4: /fan1/PWM -> Net-(M2-PWM)
- M3 pad 4: /fan2/PWM -> Net-(M3-PWM)
- M4 pad 4: /fan3/PWM -> Net-(M4-PWM)
- Q2 pad 2: unconnected-(Q2-G-Pad2) -> /fan/PWM
- Q2 pad 3: /fan/PWM -> Net-(M1-PWM)
- Q4 pad 2: unconnected-(Q4-G-Pad2) -> /fan1/PWM
- Q4 pad 3: /fan1/PWM -> Net-(M2-PWM)
- Q6 pad 2: unconnected-(Q6-G-Pad2) -> /fan2/PWM
- Q6 pad 3: /fan2/PWM -> Net-(M3-PWM)
- Q8 pad 2: unconnected-(Q8-G-Pad2) -> /fan3/PWM
- Q8 pad 3: /fan3/PWM -> Net-(M4-PWM)
- R3 pad 2: /fan/PWM -> Net-(M1-PWM)
- R5 pad 2: /fan1/PWM -> Net-(M2-PWM)
- R7 pad 2: /fan2/PWM -> Net-(M3-PWM)
- R9 pad 2: /fan3/PWM -> Net-(M4-PWM)
Routing:
- net SCL: track 0.00 -> 70.1 mm
- net SDA: track 0.00 -> 68.8 mm
- net Net-(U1-XTAL2/PB7): track 0.00 -> 33.3 mm
- net Net-(U1-XTAL1/PB6): track 0.00 -> 30.9 mm
- net RESET: track 0.00 -> 23.1 mm, vias 0 -> 1
- net SCK: track 0.00 -> 2.53 mm, vias 0 -> 1
- net /fan1/TACHO: track 0.00 -> 2.53 mm, vias 0 -> 1

Commit message: Finished PCB
Parts:
- moved D2 29.1 mm to (110.7, 149.9), turned to 180 degrees
- moved D1 24.9 mm to (104.8, 144.1)
- moved R12 22.9 mm to (110.7, 144.1)
- moved R13 22.1 mm to (110.9, 154.9)
- moved C5 14.2 mm to (124.5, 152.1), turned to -90 degrees
- moved C3 13.6 mm to (145.4, 150.8), turned to -90 degrees
- moved M3 1.27 mm to (155.6, 110.5)
- moved Q5 1.27 mm to (143.5, 119.4)
- moved R6 1.27 mm to (150.5, 103.5)
- moved Q6 1.27 mm to (143.5, 109.6)
- moved R7 1.27 mm to (150.5, 106.8)
Routing:
- net GND: track 0.00 -> 332.8 mm, vias 0 -> 19
- net VCC: track 0.00 -> 264.8 mm, vias 0 -> 11
- net +12V: track 0.00 -> 234.3 mm, vias 0 -> 12
- net /fan2/TACHO: track 0.00 -> 115.1 mm, vias 0 -> 8
- net /fan2/PWM: track 0.00 -> 109.4 mm, vias 0 -> 8
- net /fan3/TACHO: track 0.00 -> 106.9 mm, vias 0 -> 3
- net MISO: track 0.00 -> 98.2 mm, vias 0 -> 2
- net RESET: track 23.1 -> 110.3 mm, vias 1 -> 5
- net /fan3/PWM: track 0.00 -> 81.5 mm, vias 0 -> 4
- net MOSI: track 0.00 -> 64.7 mm, vias 0 -> 2
- net SCK: track 2.53 -> 66.3 mm, vias 1 -> 2
- net /fan/PWM: track 0.00 -> 63.8 mm, vias 0 -> 4
- net /fan/TACHO: track 0.00 -> 55.3 mm, vias 0 -> 2
- net /fan1/PWM: track 0.00 -> 45.7 mm, vias 0 -> 2
- net /fan1/TACHO: track 2.53 -> 47.6 mm, vias 1 -> 2
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
Commit message: revA
Parts:
- removed Q5, Q6, Q7, Q8: 2N7000, Package_TO_SOT_THT:TO-92_Inline
- removed the REF** at (101.6, 152.4)
- removed the REF** at (101.6, 76.2)
- removed the REF** at (152.4, 76.2)
- removed the REF** at (152.4, 152.4)
- added G***: LOGO, footprints:logo, F.Cu at (111.8, 96.5)
- added Q10: 2N7002, Package_TO_SOT_SMD:SOT-23, F.Cu at (83.8, 87.6)
- added Q11: 2N7002, Package_TO_SOT_SMD:SOT-23, F.Cu at (119.4, 87.6)
- added Q12: 2N7002, Package_TO_SOT_SMD:SOT-23, F.Cu at (119.4, 62.2)
- added Q9: 2N7002, Package_TO_SOT_SMD:SOT-23, F.Cu at (83.8, 62.2)
- added REF**: MountingHole_3.2mm_M3, MountingHole:MountingHole_3.2mm_M3, F.Cu at (76.2, 127.0)
- added REF**: MountingHole_3.2mm_M3, MountingHole:MountingHole_3.2mm_M3, F.Cu at (76.2, 50.8)
- added REF**: MountingHole_3.2mm_M3, MountingHole:MountingHole_3.2mm_M3, F.Cu at (127.0, 127.0)
- added REF**: MountingHole_3.2mm_M3, MountingHole:MountingHole_3.2mm_M3, F.Cu at (127.0, 50.8)
- added REF**: OSHW-Logo2_14.6x12mm_SilkScreen, Symbol:OSHW-Logo2_14.6x12mm_SilkScreen, B.Cu at (89.5, 77.5)
- Q1, Q2, Q3, Q4: value 2N7000 -> 2N7002; footprint Package_TO_SOT_THT:TO-92_Inline -> Package_TO_SOT_SMD:SOT-23
- moved C5 100.1 mm to (92.7, 57.1), turned to 180 degrees
- moved Q4 53.6 mm to (119.4, 68.6), turned to 90 degrees
- moved R3 46.9 mm to (78.7, 66.0), turned to -90 degrees
- moved R2 46.6 mm to (83.8, 57.1), turned to -90 degrees
- moved R5 41.5 mm to (78.7, 91.4), turned to -90 degrees
- moved R4 41.3 mm to (83.8, 82.5), turned to -90 degrees
- moved SW1 41.1 mm to (101.6, 61.0)
- moved C3 40.9 mm to (120.0, 118.7)
- moved R8 40.8 mm to (119.4, 57.1), turned to -90 degrees
- moved Q1 40.0 mm to (83.8, 68.6), turned to 90 degrees
- moved TP2 38.7 mm to (127.0, 105.4)
- moved TP1 38.7 mm to (127.0, 100.4)
- moved TP3 38.7 mm to (127.0, 110.5)
- moved R6 37.5 mm to (119.4, 82.5), turned to -90 degrees
- moved J1 35.9 mm to (114.9, 127.0)
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Connections:
- Q1 pad 1: GND -> /fan/PWM
- Q1 pad 2: Net-(M1-Tacho) -> GND
- Q1 pad 3: /fan/TACHO -> Net-(M1-PWM)
- Q2 pad 1: GND -> /fan1/PWM
- Q2 pad 2: /fan/PWM -> GND
- Q2 pad 3: Net-(M1-PWM) -> Net-(M2-PWM)
- Q3 pad 1: GND -> /fan2/PWM
- Q3 pad 2: Net-(M2-Tacho) -> GND
- Q3 pad 3: /fan1/TACHO -> Net-(M3-PWM)
- Q4 pad 1: GND -> /fan3/PWM
- Q4 pad 2: /fan1/PWM -> GND
- Q4 pad 3: Net-(M2-PWM) -> Net-(M4-PWM)
Routing:
- net GND: track 332.8 -> 0.00 mm, vias 19 -> 0
- net RESET: track 110.3 -> 47.4 mm, vias 5 -> 0
- net /fan2/TACHO: track 115.1 -> 53.0 mm, vias 8 -> 1
- net /fan3/TACHO: track 106.9 -> 50.7 mm, vias 3 -> 1
- net VCC: track 264.8 -> 210.2 mm, vias 11 -> 4
- net /fan2/PWM: track 109.4 -> 58.9 mm, vias 8 -> 1
- net MISO: track 98.2 -> 54.0 mm, vias 2 -> 0
- net +12V: track 234.3 -> 261.5 mm, vias 12 -> 0
- net Net-(M3-PWM): track 36.6 -> 11.3 mm, vias 4 -> 0
- net Net-(M1-PWM): track 31.3 -> 11.3 mm, vias 2 -> 0
- net MOSI: track 64.7 -> 51.9 mm, vias 2 -> 0
- net Net-(M2-PWM): track 23.3 -> 11.3 mm, vias 1 -> 0
- net Net-(M4-Tacho): track 24.8 -> 13.4 mm, vias 2 -> 0
- net /fan1/TACHO: track 47.6 -> 58.6 mm, vias 2 -> 4
- net SCL: track 66.7 -> 77.1 mm
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- added copper zone on B.Cu, net GND
- added copper zone on F.Cu, net GND
Other:
- board text added: "+12 GND"
- board text added: "I2C"
- board text added: "MULTIFAN I2C CONTROLLER"
- board text added: "PWR"
- board text added: "SCL SDA VCC GND"
- board text added: "https://github.com/ uw-madison-chem-shops/ multifan-i2c-controller"
